File: DevilsTriangle/DevilsTriangle.kicad_pcb (KiCad board)
At the start: 2 copper layers, 89.4 x 67.7 mm, 51 parts, among them SW1 SPST, SW2 SPST, SW3 SPST, SW4 SPST, U1 LM324N, U2 LM324N, U3 LM324N

Commit message: more silkscreen
Parts:
- added G***: LOGO, kicad-cbase:c-base-logo-ceva, F.Cu at (171.3, 85.3)
- added G***: LOGO, kicad-cbase:c-base, F.Cu at (175.7, 103.6)
