File: SchrittMacher/ClockGenerator.sch (KiCad schematic (older format))
At the start: 5 parts, among them U3 LM555N

Commit message: fixed some circuit problems in schrittmacher
Parts:
- RV1: symbol POT -> POT-RESCUE-SchrittMacher
Connections:
- net GND: no longer RV1.3
- net at C2.1, U3.2 (TR), U3.6 (THR): now also RV1.3; no longer RV1.2
- net at R5.2, RV1.1, U3.7 (DIS): now also RV1.2
Other:
- moved on the sheet: C2
Changed lines of the file:
@@
 EESchema Schematic File Version 2
+LIBS:SchrittMacher-rescue
 LIBS:power
 LIBS:device
@@
 $EndComp
 $Comp
-L POT RV1
+L POT-RESCUE-SchrittMacher RV1
 U 1 1 56EA9787
 P 4700 2600
@@
 	3950 2400 4700 2400
 Wire Wire Line
-	3950 2600 4550 2600
-Wire Wire Line
 	4700 2350 4700 2450
 Connection ~ 4700 2400
@@
 	2950 2600 2850 2600
 Wire Wire Line
-	4700 2750 4700 3300
-Wire Wire Line
-	4300 2600 4300 2800
-Connection ~ 4300 2600
-Wire Wire Line
-	4300 3100 4300 3200
-Wire Wire Line
-	4300 3200 4700 3200
-Connection ~ 4700 3200
-Wire Wire Line
 	2950 2400 2650 2400
 Wire Wire Line
@@
 Wire Wire Line
 	4050 3200 4050 2600
-Connection ~ 4050 2600
 Wire Wire Line
 	2650 2950 2650 2850
@@
 L CP C2
 U 1 1 5710E7C6
-P 4300 2950
-F 0 "C2" H 4325 3050 50  0000 L CNN
-F 1 "2.2uF" H 4325 2850 50  0000 L CNN
-F 2 "Capacitors_ThroughHole:C_Radial_D5_L6_P2.5" H 4338 2800 50  0001 C CNN
-F 3 "" H 4300 2950 50  0000 C CNN
-	1    4300 2950
-	1    0    0    -1
-$EndComp
+P 4700 3050
+F 0 "C2" H 4725 3150 50  0000 L CNN
+F 1 "2.2uF" H 4725 2950 50  0000 L CNN
+F 2 "Capacitors_ThroughHole:C_Radial_D5_L6_P2.5" H 4738 2900 50  0001 C CNN
+F 3 "" H 4700 3050 50  0000 C CNN
+	1    4700 3050
+	1    0    0    -1
+$EndComp
+Wire Wire Line
+	4550 2600 4550 2400
+Connection ~ 4550 2400
+Wire Wire Line
+	4700 3300 4700 3200
+Wire Wire Line
+	4700 2900 4700 2750
+Wire Wire Line
+	4700 2800 4050 2800
+Connection ~ 4050 2800
+Connection ~ 4700 2800
+Wire Wire Line
+	4050 2600 3950 2600
 $EndSCHEMATC
