File: SchrittMacher/SchrittMacher.sch (KiCad schematic (older format))
At the start: 15 parts, among them CON1 BARREL_JACK, J1 JACK_2P, J2 JACK_2P, J3 JACK_2P, J4 JACK_2P, SW1 SPST, SW2 SPST, U1 TL072, U2 4017

Commit message: fixed some circuit problems in schrittmacher
Connections:
- net +12V: now also U2.16 (VDD); no longer U2.8 (VSS)
- net GND: now also U2.8 (VSS); no longer U2.16 (VDD)
Changed lines of the file:
@@
 EESchema Schematic File Version 2
+LIBS:SchrittMacher-rescue
 LIBS:power
 LIBS:device
@@
 L GND #PWR011
 U 1 1 570C595D
-P 4550 2350
-F 0 "#PWR011" H 4550 2100 50  0001 C CNN
-F 1 "GND" H 4550 2200 50  0000 C CNN
-F 2 "" H 4550 2350 50  0000 C CNN
-F 3 "" H 4550 2350 50  0000 C CNN
-	1    4550 2350
-	1    0    0    -1
-$EndComp
-Text GLabel 4550 900  1    60   Input ~ 0
+P 4550 900
+F 0 "#PWR011" H 4550 650 50  0001 C CNN
+F 1 "GND" H 4550 750 50  0000 C CNN
+F 2 "" H 4550 900 50  0000 C CNN
+F 3 "" H 4550 900 50  0000 C CNN
+	1    4550 900
+	-1   0    0    1
+$EndComp
+Text GLabel 4550 2350 3    60   Input ~ 0
 VCC
 Wire Wire Line
