File: SchrittMacher/Steps.sch (KiCad schematic (older format))
At the start: 70 parts, among them Q1 BC547, Q10 BC547, Q2 BC547, Q3 BC547, Q4 BC547, Q5 BC547, Q6 BC547, Q7 BC547, Q8 BC547, Q9 BC547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

Commit message: fixed some circuit problems in schrittmacher
Parts:
- D1, D11, D12, D13, D14, D15, D2, D3, D4, D5: symbol LED -> LED-RESCUE-SchrittMacher
- RV10, RV11, RV2, RV3, RV4, RV5, RV6, RV7, RV8, RV9: symbol POT -> POT-RESCUE-SchrittMacher
Connections:
- net at D8.1 (K), SW5.2: no longer R11.2
- net at RV4.3, SW5.1: now also R11.2
- net at D9.1 (K), SW6.2: no longer R13.2
- net at RV5.3, SW6.1: now also R13.2
- net at D10.1 (K), SW7.2: no longer R15.2
- net at RV6.3, SW7.1: now also R15.2
- net at D16.1 (K), SW8.2: no longer R17.2
- net at RV7.3, SW8.1: now also R17.2
- net at D17.1 (K), SW9.2: no longer R19.2
- net at RV8.3, SW9.1: now also R19.2
- net at D18.1 (K), SW10.2: no longer R21.2
- net at RV9.3, SW10.1: now also R21.2
- net at D19.1 (K), SW11.2: no longer R23.2
- net at RV10.3, SW11.1: now also R23.2
- net at D20.1 (K), SW12.2: no longer R25.2
- net at RV11.3, SW12.1: now also R25.2
- net at D6.1 (K), SW3.2: no longer R7.2
- net at RV2.3, SW3.1: now also R7.2
- net at D7.1 (K), SW4.2: no longer R9.2
- net at RV3.3, SW4.1: now also R9.2
Changed lines of the file:
@@
 EESchema Schematic File Version 2
+LIBS:SchrittMacher-rescue
 LIBS:power
 LIBS:device
@@
 $EndDescr
 $Comp
-L LED D1
+L LED-RESCUE-SchrittMacher D1
 U 1 1 56E91BB6
 P 950 1100
+AR Path="/56E91BB6" Ref="D1"  Part="1"
+AR Path="/56E7296A/56E91BB6" Ref="D1"  Part="1"
 F 0 "D1" H 950 1200 50  0000 C CNN
 F 1 "LED" H 950 1000 50  0000 C CNN
@@
 F 3 "" H 1250 2400 50  0000 C CNN
 	1    1250 2400
-	0    1    1    0
-$EndComp
-Wire Wire Line
-	1250 2150 1250 2250
-Wire Wire Line
-	1450 2200 1250 2200
-Connection ~ 1250 2200
-$Comp
-L POT RV2
+	0    -1   1    0
+$EndComp
+$Comp
+L POT-RESCUE-SchrittMacher RV2
 U 1 1 56E91BE0
 P 1450 1300
@@
 $EndComp
 Wire Wire Line
-	1450 2200 1450 2800
-Wire Wire Line
 	1450 2800 1750 2800
 Wire Wire Line
 	1450 1800 1650 1800
 Wire Wire Line
-	1450 1450 1450 1800
+	1450 1450 1450 2150
 Wire Wire Line
 	1600 1300 1650 1300
@@
 RESET
 $Comp
-L LED D2
+L LED-RESCUE-SchrittMacher D2
 U 1 1 56EA46BA
 P 2600 1100
+AR Path="/56EA46BA" Ref="D2"  Part="1"
+AR Path="/56E7296A/56EA46BA" Ref="D2"  Part="1"
 F 0 "D2" H 2600 1200 50  0000 C CNN
 F 1 "LED" H 2600 1000 50  0000 C CNN
@@
 	0    1    1    0
 $EndComp
-Wire Wire Line
-	2900 2150 2900 2250
-Wire Wire Line
-	3100 2200 2900 2200
-Connection ~ 2900 2200
-$Comp
-L POT RV3
+$Comp
+L POT-RESCUE-SchrittMacher RV3
 U 1 1 56EA46DE
 P 3100 1300
@@
 $EndComp
 Wire Wire Line
-	3100 2200 3100 2800
-Wire Wire Line
 	3100 2800 3400 2800
 Wire Wire Line
 	3100 1800 3300 1800
 Wire Wire Line
-	3100 1450 3100 1800
+	3100 1450 3100 2150
 Wire Wire Line
 	3250 1300 3300 1300
@@
 	2600 900  2600 850
 $Comp
-L LED D3
+L LED-RESCUE-SchrittMacher D3
 U 1 1 56E7157F
 P 4300 1100
+AR Path="/56E7157F" Ref="D3"  Part="1"
+AR Path="/56E7296A/56E7157F" Ref="D3"  Part="1"
 F 0 "D3" H 4300 1200 50  0000 C CNN
 F 1 "LED" H 4300 1000 50  0000 C CNN
@@
 	0    1    1    0
 $EndComp
-Wire Wire Line
-	4600 2150 4600 2250
-Wire Wire Line
-	4800 2200 4600 2200
-Connection ~ 4600 2200
-$Comp
-L POT RV4
+$Comp
+L POT-RESCUE-SchrittMacher RV4
 U 1 1 56E715A3
 P 4800 1300
@@
 $EndComp
 Wire Wire Line
-	4800 2200 4800 2800
-Wire Wire Line
 	4800 2800 5100 2800
 Wire Wire Line
 	4800 1800 5000 1800
 Wire Wire Line
-	4800 1450 4800 1800
+	4800 1450 4800 2150
 Wire Wire Line
 	4950 1300 5000 1300
@@
 	4300 900  4300 850
 $Comp
-L LED D4
+L LED-RESCUE-SchrittMacher D4
 U 1 1 56E82BAC
 P 6000 1100
+AR Path="/56E82BAC" Ref="D4"  Part="1"
+AR Path="/56E7296A/56E82BAC" Ref="D4"  Part="1"
 F 0 "D4" H 6000 1200 50  0000 C CNN
 F 1 "LED" H 6000 1000 50  0000 C CNN
@@
 	0    1    1    0
 $EndComp
-Wire Wire Line
-	6300 2150 6300 2250
-Wire Wire Line
-	6500 2200 6300 2200
-Connection ~ 6300 2200
-$Comp
-L POT RV5
+$Comp
+L POT-RESCUE-SchrittMacher RV5
 U 1 1 56E82BD5
 P 6500 1300
@@
 $EndComp
 Wire Wire Line
-	6500 2200 6500 2800
-Wire Wire Line
 	6500 2800 6800 2800
 Wire Wire Line
 	6500 1800 6700 1800
 Wire Wire Line
-	6500 1450 6500 1800
+	6500 1450 6500 2150
 Wire Wire Line
 	6650 1300 6700 1300
@@
 	6000 900  6000 850
 $Comp
-L LED D5
+L LED-RESCUE-SchrittMacher D5
 U 1 1 56E82EF2
 P 7700 1100
+AR Path="/56E82EF2" Ref="D5"  Part="1"
+AR Path="/56E7296A/56E82EF2" Ref="D5"  Part="1"
 F 0 "D5" H 7700 1200 50  0000 C CNN
 F 1 "LED" H 7700 1000 50  0000 C CNN
@@
 	0    1    1    0
 $EndComp
-Wire Wire Line
-	8000 2150 8000 2250
-Wire Wire Line
-	8200 2200 8000 2200
-Connection ~ 8000 2200
-$Comp
-L POT RV6
+$Comp
+L POT-RESCUE-SchrittMacher RV6
 U 1 1 56E82F1B
 P 8200 1300
@@
 $EndComp
 Wire Wire Line
-	8200 2200 8200 2800
-Wire Wire Line
 	8200 2800 8500 2800
 Wire Wire Line
 	8200 1800 8400 1800
 Wire Wire Line
-	8200 1450 8200 1800
+	8200 1450 8200 2150
 Wire Wire Line
 	8350 1300 8400 1300
@@
 	7700 900  7700 850
 $Comp
-L LED D11
+L LED-RESCUE-SchrittMacher D11
 U 1 1 56E839E7
 P 900 3900
+AR Path="/56E839E7" Ref="D11"  Part="1"
+AR Path="/56E7296A/56E839E7" Ref="D11"  Part="1"
 F 0 "D11" H 900 4000 50  0000 C CNN
 F 1 "LED" H 900 3800 50  0000 C CNN
@@
 	0    1    1    0
 $EndComp
-Wire Wire Line
-	1200 4950 1200 5050
-Wire Wire Line
-	1400 5000 1200 5000
-Connection ~ 1200 5000
-$Comp
-L POT RV7
+$Comp
+L POT-RESCUE-SchrittMacher RV7
 U 1 1 56E83A10
 P 1400 4100
@@
 $EndComp
 Wire Wire Line
-	1400 5000 1400 5600
-Wire Wire Line
 	1400 5600 1700 5600
 Wire Wire Line
 	1400 4600 1600 4600
 Wire Wire Line
-	1400 4250 1400 4600
+	1400 4250 1400 4950
 Wire Wire Line
 	1550 4100 1600 4100
@@
 	900  3700 900  3650
 $Comp
-L LED D12
+L LED-RESCUE-SchrittMacher D12
 U 1 1 56E83EFB
 P 2600 3900
+AR Path="/56E83EFB" Ref="D12"  Part="1"
+AR Path="/56E7296A/56E83EFB" Ref="D12"  Part="1"
 F 0 "D12" H 2600 4000 50  0000 C CNN
 F 1 "LED" H 2600 3800 50  0000 C CNN
@@
 	0    1    1    0
 $EndComp
-Wire Wire Line
-	2900 4950 2900 5050
-Wire Wire Line
-	3100 5000 2900 5000
-Connection ~ 2900 5000
-$Comp
-L POT RV8
+$Comp
+L POT-RESCUE-SchrittMacher RV8
 U 1 1 56E83F24
 P 3100 4100
@@
 $EndComp
 Wire Wire Line
-	3100 5000 3100 5600
-Wire Wire Line
 	3100 5600 3400 5600
 Wire Wire Line
 	3100 4600 3300 4600
 Wire Wire Line
-	3100 4250 3100 4600
+	3100 4250 3100 4950
 Wire Wire Line
 	3250 4100 3300 4100
@@
 	2600 3700 2600 3650
 $Comp
-L LED D13
+L LED-RESCUE-SchrittMacher D13
 U 1 1 56E84416
 P 4300 3900
+AR Path="/56E84416" Ref="D13"  Part="1"
+AR Path="/56E7296A/56E84416" Ref="D13"  Part="1"
 F 0 "D13" H 4300 4000 50  0000 C CNN
 F 1 "LED" H 4300 3800 50  0000 C CNN
@@
 	0    1    1    0
 $EndComp
-Wire Wire Line
-	4600 4950 4600 5050
-Wire Wire Line
-	4800 5000 4600 5000
-Connection ~ 4600 5000
-$Comp
-L POT RV9
+$Comp
+L POT-RESCUE-SchrittMacher RV9
 U 1 1 56E8443F
 P 4800 4100
@@
 $EndComp
 Wire Wire Line
-	4800 5000 4800 5600
-Wire Wire Line
 	4800 5600 5100 5600
 Wire Wire Line
 	4800 4600 5000 4600
 Wire Wire Line
-	4800 4250 4800 4600
+	4800 4250 4800 4950
 Wire Wire Line
 	4950 4100 5000 4100
@@
 	4300 3700 4300 3650
 $Comp
-L LED D14
+L LED-RESCUE-SchrittMacher D14
 U 1 1 56E849EE
 P 6000 3900
+AR Path="/56E849EE" Ref="D14"  Part="1"
+AR Path="/56E7296A/56E849EE" Ref="D14"  Part="1"
 F 0 "D14" H 6000 4000 50  0000 C CNN
 F 1 "LED" H 6000 3800 50  0000 C CNN
@@
 	0    1    1    0
 $EndComp
-Wire Wire Line
-	6300 4950 6300 5050
-Wire Wire Line
-	6500 5000 6300 5000
-Connection ~ 6300 5000
-$Comp
-L POT RV10
+$Comp
+L POT-RESCUE-SchrittMacher RV10
 U 1 1 56E84A17
 P 6500 4100
@@
 $EndComp
 Wire Wire Line
-	6500 5000 6500 5600
-Wire Wire Line
 	6500 5600 6800 5600
 Wire Wire Line
 	6500 4600 6700 4600
 Wire Wire Line
-	6500 4250 6500 4600
+	6500 4250 6500 4950
 Wire Wire Line
 	6650 4100 6700 4100
@@
 	6000 3700 6000 3650
 $Comp
-L LED D15
+L LED-RESCUE-SchrittMacher D15
 U 1 1 56E852B3
 P 7700 3900
+AR Path="/56E852B3" Ref="D15"  Part="1"
+AR Path="/56E7296A/56E852B3" Ref="D15"  Part="1"
 F 0 "D15" H 7700 4000 50  0000 C CNN
 F 1 "LED" H 7700 3800 50  0000 C CNN
@@
 	0    1    1    0
 $EndComp
-Wire Wire Line
-	8000 4950 8000 5050
-Wire Wire Line
-	8200 5000 8000 5000
-Connection ~ 8000 5000
-$Comp
-L POT RV11
+$Comp
+L POT-RESCUE-SchrittMacher RV11
 U 1 1 56E852DC
 P 8200 4100
@@
 $EndComp
 Wire Wire Line
-	8200 5000 8200 5600
-Wire Wire Line
 	8200 5600 8500 5600
 Wire Wire Line
 	8200 4600 8400 4600
 Wire Wire Line
-	8200 4250 8200 4600
+	8200 4250 8200 4950
 Wire Wire Line
 	8350 4100 8400 4100
@@
 Wire Wire Line
 	900  4650 900  4600
+Wire Wire Line
+	1250 2250 1450 2250
+Wire Wire Line
+	1450 2250 1450 2800
+Wire Wire Line
+	1450 2150 1250 2150
+Connection ~ 1450 1800
+Wire Wire Line
+	2900 2250 3100 2250
+Wire Wire Line
+	3100 2250 3100 2800
+Wire Wire Line
+	3100 2150 2900 2150
+Connection ~ 3100 1800
+Wire Wire Line
+	4800 2800 4800 2250
+Wire Wire Line
+	4800 2250 4600 2250
+Wire Wire Line
+	4800 2150 4600 2150
+Connection ~ 4800 1800
+Wire Wire Line
+	6300 2250 6500 2250
+Wire Wire Line
+	6500 2250 6500 2800
+Wire Wire Line
+	6500 2150 6300 2150
+Connection ~ 6500 1800
+Wire Wire Line
+	8000 2250 8200 2250
+Wire Wire Line
+	8200 2250 8200 2800
+Wire Wire Line
+	8200 2150 8000 2150
+Connection ~ 8200 1800
+Wire Wire Line
+	1200 5050 1400 5050
+Wire Wire Line
+	1400 5050 1400 5600
+Wire Wire Line
+	1400 4950 1200 4950
+Connection ~ 1400 4600
+Wire Wire Line
+	2900 5050 3100 5050
+Wire Wire Line
+	3100 5050 3100 5600
+Wire Wire Line
+	3100 4950 2900 4950
+Connection ~ 3100 4600
+Wire Wire Line
+	4600 5050 4800 5050
+Wire Wire Line
+	4800 5050 4800 5600
+Wire Wire Line
+	4800 4950 4600 4950
+Connection ~ 4800 4600
+Wire Wire Line
+	6300 5050 6500 5050
+Wire Wire Line
+	6500 5050 6500 5600
+Wire Wire Line
+	6500 4950 6300 4950
+Connection ~ 6500 4600
+Wire Wire Line
+	8000 5050 8200 5050
+Wire Wire Line
+	8200 5050 8200 5600
+Wire Wire Line
+	8200 4950 8000 4950
+Connection ~ 8200 4600
 $EndSCHEMATC
